File: board/dc-motor-driver-adapter.kicad_pcb (KiCad board)
At the start: 2 copper layers, 21 x 15 mm, 16 parts, among them J1 Conn_01x03, J2 Conn_01x03, Q1 BC817-40, Q2 BC817-40, U1 CH32V003J4M6, U2 MCP4725A0T-E/CH

Commit message: Плата замовлена.
Parts:
- moved R2 0.25 mm to (165.3, 107.6)
- moved R5 0.15 mm to (168.4, 107.6)
Routing:
- net +5V: track 31.2 -> 32.5 mm
- net GND: track 11.8 -> 12.2 mm, vias 10 -> 12
Other:
- board text added: "+5V"
- board text added: "FRW"
- board text added: "GND"
- board text added: "PWM"
- board text added: "RRW"
- board text added: "SPD"
- board text added: "SWIO"
