File: board/revision-1/dc-motor-driver-adapter.kicad_sch (KiCad schematic)
At the start: 16 parts, among them J1 Conn_01x03, J2 Conn_01x03, Q1 BC817-40, Q2 BC817-40, U1 CH32V003J4M6, U2 MCP4725A0T-E/CH

Commit message: Збереження.
Other:
- note added: "3. PA2, T1CH2N, 7. PC4, T1CH4, T1CH1CH2N 5. PC1, T2CH4 6. PC2, T2CH2"
- note added: "Альтернативні функції виводів контролера CH32V003J4M6"
- moved on the sheet: FID1, FID2
Changed lines of the file:
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@@
+		)
+	)
+	(text "3. PA2, T1CH2N, \n7. PC4, T1CH4, T1CH1CH2N\n\n5. PC1, T2CH4\n6. PC2, T2CH2"
+		(exclude_from_sim no)
+		(at 82.804 156.464 0)
+		(effects
+			(font
+				(size 1.27 1.27)
+			)
+			(justify left)
+		)
+	)
+	(text "Альтернативні функції виводів контролера CH32V003J4M6"
+		(exclude_from_sim no)
+		(at 112.014 147.066 0)
+		(effects
+			(font
+				(size 1.27 1.27)
+			)
 		)
 	)
@@
 	(symbol
 		(lib_id "Mechanical:Fiducial")
-		(at 50.8 172.72 0)
+		(at 17.78 177.8 0)
 		(unit 1)
 		(exclude_from_sim yes)
@@
 		(fields_autoplaced yes)
 		(property "Reference" "FID1"
-			(at 53.34 171.4499 0)
+			(at 20.32 176.5299 0)
 			(effects
 				(font
@@
 		)
 		(property "Value" "Fiducial"
-			(at 53.34 173.9899 0)
+			(at 20.32 179.0699 0)
 			(effects
 				(font
@@
 		)
 		(property "Footprint" "Fiducial:Fiducial_1mm_Mask2mm"
-			(at 50.8 172.72 0)
+			(at 17.78 177.8 0)
 			(effects
 				(font
@@
 		)
 		(property "Datasheet" "~"
-			(at 50.8 172.72 0)
+			(at 17.78 177.8 0)
 			(effects
 				(font
@@
 		)
 		(property "Description" "Fiducial Marker"
-			(at 50.8 172.72 0)
+			(at 17.78 177.8 0)
 			(effects
 				(font
@@
 	(symbol
 		(lib_id "Mechanical:Fiducial")
-		(at 69.85 172.72 0)
+		(at 36.83 177.8 0)
 		(unit 1)
 		(exclude_from_sim yes)
@@
 		(fields_autoplaced yes)
 		(property "Reference" "FID2"
-			(at 72.39 171.4499 0)
+			(at 39.37 176.5299 0)
 			(effects
 				(font
@@
 		)
 		(property "Value" "Fiducial"
-			(at 72.39 173.9899 0)
+			(at 39.37 179.0699 0)
 			(effects
 				(font
@@
 		)
 		(property "Footprint" "Fiducial:Fiducial_1mm_Mask2mm"
-			(at 69.85 172.72 0)
+			(at 36.83 177.8 0)
 			(effects
 				(font
@@
 		)
 		(property "Datasheet" "~"
-			(at 69.85 172.72 0)
+			(at 36.83 177.8 0)
 			(effects
 				(font
@@
 		)
 		(property "Description" "Fiducial Marker"
-			(at 69.85 172.72 0)
-			(effects
-				(font
+			(at 36.83 177.8 0)
+			(effects
+				(font
